Commit message: added urdf and launch files

File: description/robot.urdf.xacro (robot description, xacro)
@@ -1,16 +1,98 @@
 <?xml version="1.0"?>
 <robot xmlns:xacro="https://www.ros.org/wiki/xacro" name="robot">
+    <material name="white">
+        <color rgba="1.0 1.0 1.0 1.0"/>
+    </material>
+    <material name="red">
+        <color rgba="1.0 0.0 0.0 1.0"/>
+    </material>
+    <material name="green">
+        <color rgba="0.0 1.0 0.0 1.0"/>
+    </material>
+    <material name="blue">
+        <color rgba="0.0 0.0 1.0 1.0"/>
+    </material>
     <link name="base_link"></link>
     <joint name="chassis_joint" type="fixed">
         <parent link="base_link"/>
         <child link="chassis"/>
-        <origin xyz="0.0 0.0 0.0" rpy="0.0 0.0 0.0"/>
+        <origin xyz="0.0 0.0 0.065" rpy="0.0 0.0 0.0"/>
     </joint>
     <link name="chassis">
         <visual>
-            <origin xyz="0.0 0.0 0.075" rpy="0.0 0.0 0.0"/>
+            <origin xyz="0.0 0.0 0.0" rpy="0.0 0.0 0.0"/>
             <geometry>
-                <box size="0.3 0.2 0.15"/>
+                <box size="0.3 0.2 0.05"/>
             </geometry>
+            <material name="white"/>
+        </visual>
+    </link>
+    <joint name="left_wheel_1_joint" type="continuous">
+        <parent link="base_link"/>
+        <child link="left_wheel_1"/>
+        <origin xyz="0.075 0.115 0.05" rpy="-${pi/2} 0.0 0.0"/>
+        <axis xyz="0.0 0.0 1.0"/>
+    </joint>
+    <link name="left_wheel_1">
+        <visual>
+            <geometry>
+                <cylinder radius="0.05" length="0.03"/>
+            </geometry>
+            <material name="blue"/>
+        </visual>
+    </link>
+    <joint name="left_wheel_2_joint" type="continuous">
+        <parent link="base_link"/>
+        <child link="left_wheel_2"/>
+        <origin xyz="-0.075 0.115 0.05" rpy="-${pi/2} 0.0 0.0"/>
+        <axis xyz="0.0 0.0 1.0"/>
+    </joint>
+    <link name="left_wheel_2">
+        <visual>
+            <geometry>
+                <cylinder radius="0.05" length="0.03"/>
+            </geometry>
+            <material name="blue"/>
+        </visual>
+    </link>
+    <joint name="right_wheel_1_joint" type="continuous">
+        <parent link="base_link"/>
+        <child link="right_wheel_1"/>
+        <origin xyz="0.075 -0.115 0.05" rpy="${pi/2} 0.0 0.0"/>
+        <axis xyz="0.0 0.0 -1.0"/>
+    </joint>
+    <link name="right_wheel_1">
+        <visual>
+            <geometry>
+                <cylinder radius="0.05" length="0.03"/>
+            </geometry>
+            <material name="blue"/>
+        </visual>
+    </link>
+    <joint name="right_wheel_2_joint" type="continuous">
+        <parent link="base_link"/>
+        <child link="right_wheel_2"/>
+        <origin xyz="-0.075 -0.115 0.05" rpy="${pi/2} 0.0 0.0"/>
+        <axis xyz="0.0 0.0 -1.0"/>
+    </joint>
+    <link name="right_wheel_2">
+        <visual>
+            <geometry>
+                <cylinder radius="0.05" length="0.03"/>
+            </geometry>
+            <material name="blue"/>
+        </visual>
+    </link>
+    <joint name='lidar_link' type="fixed">
+        <parent link="base_link"/>
+        <child link="lidar"/>
+        <origin xyz="0.075 0.0 0.105" rpy="0.0 0.0 0.0"/>
+    </joint>
+    <link name="lidar">
+        <visual>
+            <geometry>
+                <cylinder radius="0.05" length="0.03"/>
+            </geometry>
+            <material name="red"/>
         </visual>
     </link>

Commit message: added keypress control to gazebo simulation

File: description/robot.urdf.xacro (robot description, xacro)
@@ -1,4 +1,29 @@
 <?xml version="1.0"?>
 <robot xmlns:xacro="https://www.ros.org/wiki/xacro" name="robot">
+    <xacro:macro name="inertial_box" params="mass x y z *origin">
+        <inertial>
+            <xacro:insert_block name="origin"/>
+            <mass value="${mass}"/>
+            <inertia ixx="${(1/12) * mass * (y*y + z*z)}" ixy="0.0" ixz="0.0" iyy="${(1/12) * mass * (x*x + z*z)}" iyz="0.0" izz="${(1/12) * mass * (x*x + y*y)}"/>
+        </inertial>
+    </xacro:macro>
+    <xacro:macro name="inertial_cylinder" params="mass length radius *origin">
+        <inertial>
+            <xacro:insert_block name="origin"/>
+            <mass value="${mass}" />
+            <inertia ixx="${(1/12) * mass * (3*radius*radius + length*length)}" ixy="0.0" ixz="0.0"
+                    iyy="${(1/12) * mass * (3*radius*radius + length*length)}" iyz="0.0"
+                    izz="${(1/2) * mass * (radius*radius)}" />
+        </inertial>
+    </xacro:macro>
+    <xacro:macro name="inertial_sphere" params="mass radius *origin">
+        <inertial>
+            <xacro:insert_block name="origin"/>
+            <mass value="${mass}" />
+            <inertia ixx="${(2/5) * mass * (radius*radius)}" ixy="0.0" ixz="0.0"
+                    iyy="${(2/5) * mass * (radius*radius)}" iyz="0.0"
+                    izz="${(2/5) * mass * (radius*radius)}" />
+        </inertial>
+    </xacro:macro>
     <material name="white">
         <color rgba="1.0 1.0 1.0 1.0"/>
@@ -27,4 +52,13 @@
             <material name="white"/>
         </visual>
+        <collision>
+            <origin xyz="0.0 0.0 0.0" rpy="0.0 0.0 0.0"/>
+            <geometry>
+                <box size="0.3 0.2 0.05"/>
+            </geometry>
+        </collision>
+        <xacro:inertial_box mass="0.5" x="0.3" y="0.2" z="0.15">
+            <origin xyz="0.0 0.0 0.0" rpy="0.0 0.0 0.0"/>
+        </xacro:inertial_box>
     </link>
     <joint name="left_wheel_1_joint" type="continuous">
@@ -41,4 +75,12 @@
             <material name="blue"/>
         </visual>
+        <collision>
+            <geometry>
+                <cylinder radius="0.05" length="0.03"/>
+            </geometry>
+        </collision>
+        <xacro:inertial_cylinder mass="0.05" length="0.03" radius="0.05">
+            <origin xyz="0.075 0.115 0.05" rpy="-${pi/2} 0.0 0.0"/>
+        </xacro:inertial_cylinder>
     </link>
     <joint name="left_wheel_2_joint" type="continuous">
@@ -55,4 +97,12 @@
             <material name="blue"/>
         </visual>
+        <collision>
+            <geometry>
+                <cylinder radius="0.05" length="0.03"/>
+            </geometry>
+        </collision>
+        <xacro:inertial_cylinder mass="0.05" length="0.03" radius="0.05">
+            <origin xyz="-0.075 0.115 0.05" rpy="-${pi/2} 0.0 0.0"/>
+        </xacro:inertial_cylinder>
     </link>
     <joint name="right_wheel_1_joint" type="continuous">
@@ -69,4 +119,12 @@
             <material name="blue"/>
         </visual>
+        <collision>
+            <geometry>
+                <cylinder radius="0.05" length="0.03"/>
+            </geometry>
+        </collision>
+        <xacro:inertial_cylinder mass="0.05" length="0.03" radius="0.05">
+            <origin xyz="0.075 -0.115 0.05" rpy="${pi/2} 0.0 0.0"/>
+        </xacro:inertial_cylinder>
     </link>
     <joint name="right_wheel_2_joint" type="continuous">
@@ -83,4 +141,12 @@
             <material name="blue"/>
         </visual>
+        <collision>
+            <geometry>
+                <cylinder radius="0.05" length="0.03"/>
+            </geometry>
+        </collision>
+        <xacro:inertial_cylinder mass="0.05" length="0.03" radius="0.05">
+            <origin xyz="-0.075 -0.115 0.05" rpy="${pi/2} 0.0 0.0"/>
+        </xacro:inertial_cylinder>
     </link>
     <joint name='lidar_link' type="fixed">
@@ -96,4 +162,74 @@
             <material name="red"/>
         </visual>
-    </link>
+        <collision>
+            <geometry>
+                <cylinder radius="0.05" length="0.03"/>
+            </geometry>
+        </collision>
+    </link>
+    <gazebo>
+        <plugin name="gz::sim::systems::DiffDrive" filename="gz-sim-diff-drive-system">
+            <left_joint>left_wheel_1_joint</left_joint>
+            <right_joint>right_wheel_1_joint</right_joint>
+            <left_joint>left_wheel_2_joint</left_joint>
+            <right_joint>right_wheel_2_joint</right_joint>
+            <wheel_separation>0.230</wheel_separation>
+            <wheel_radius>0.05</wheel_radius>
+            <topic>cmd_vel</topic>
+            <frame_id>odom</frame_id>
+            <child_frame_id>base_link</child_frame_id>
+            <odom_topic>odom</odom_topic>
+            <odom_publish_frequency>30</odom_publish_frequency>
+            <publish_odom>true</publish_odom>
+            <publish_odom_tf>true</publish_odom_tf>
+            <tf_topic>/tf</tf_topic>
+        </plugin>
+        <plugin name="gz::sim::systems::JointStatePublisher" filename="gz-sim-joint-state-publisher-system">
+            <topic>joint_states</topic>
+            <joint_name>left_wheel_1_joint</joint_name>
+            <joint_name>left_wheel_2_joint</joint_name>
+            <joint_name>right_wheel_1_joint</joint_name>
+            <joint_name>right_wheel_2_joint</joint_name>
+        </plugin>
+        <!-- Moving Forward-->
+        <plugin filename="gz-sim-triggered-publisher-system"
+                name="gz::sim::systems::TriggeredPublisher">
+            <input type="gz.msgs.Int32" topic="/keyboard/keypress">
+                <match field="data">16777235</match>
+            </input>
+            <output type="gz.msgs.Twist" topic="/cmd_vel">
+                linear: {x: 0.5}, angular: {z: 0.0}
+            </output>
+        </plugin>
+        <!-- Moving Backward-->
+        <plugin filename="gz-sim-triggered-publisher-system"
+                name="gz::sim::systems::TriggeredPublisher">
+            <input type="gz.msgs.Int32" topic="/keyboard/keypress">
+                <match field="data">16777237</match>
+            </input>
+            <output type="gz.msgs.Twist" topic="/cmd_vel">
+                linear: {x: -0.5}, angular: {z: 0.0}
+            </output>
+        </plugin>
+        <!-- Moving Left-->
+        <plugin filename="gz-sim-triggered-publisher-system"
+                name="gz::sim::systems::TriggeredPublisher">
+            <input type="gz.msgs.Int32" topic="/keyboard/keypress">
+                <match field="data">16777234</match>
+            </input>
+            <output type="gz.msgs.Twist" topic="/cmd_vel">
+                linear: {x: 0.0}, angular: {z: 0.5}
+            </output>
+        </plugin>
+        <!--Moving Right-->
+        <plugin filename="gz-sim-triggered-publisher-system"
+                name="gz::sim::systems::TriggeredPublisher">
+            <input type="gz.msgs.Int32" topic="/keyboard/keypress">
+                <match field="data">16777236</match>
+            </input>
+            <output type="gz.msgs.Twist" topic="/cmd_vel">
+                linear: {x: 0.0}, angular: {z: -0.5}
+            </output>
+        </plugin>
+    </gazebo>
 </robot>

Commit message: started ros2 control

File: description/robot.urdf.xacro (robot description, xacro)
@@ -1,4 +1,5 @@
 <?xml version="1.0"?>
 <robot xmlns:xacro="https://www.ros.org/wiki/xacro" name="robot">
+    <xacro:include filename="ros2_control.xacro"/>
     <xacro:macro name="inertial_box" params="mass x y z *origin">
         <inertial>
@@ -150,5 +151,5 @@
         </xacro:inertial_cylinder>
     </link>
-    <joint name='lidar_link' type="fixed">
+    <joint name="lidar_link" type="fixed">
         <parent link="base_link"/>
         <child link="lidar"/>
@@ -167,6 +168,44 @@
             </geometry>
         </collision>
-    </link>
+        <xacro:inertial_cylinder mass="0.05" length="0.03" radius="0.05">
+            <origin xyz="0.075 0.0 0.105" rpy="0.0 0.0 0.0"/>
+        </xacro:inertial_cylinder>
+    </link>
+    <gazebo reference="lidar">
+        <sensor name="lidar" type="gpu_lidar">
+            <pose relative_to="lidar_link"> 0 0 0 0 0 0 </pose>
+            <visualize>true</visualize>
+            <update_rate>10</update_rate>
+            <always_on>1</always_on>
+            <lidar>
+                <scan>
+                    <horizontal>
+                        <samples>360</samples>
+                        <min_angle>-3.14</min_angle>
+                        <max_angle>3.14</max_angle>
+                    </horizontal>
+                    <vertical>
+                        <samples>1</samples>
+                        <resolution>0.01</resolution>
+                        <min_angle>0</min_angle>
+                        <max_angle>0</max_angle>
+                    </vertical>
+                </scan>
+                <range>
+                    <min>0.3</min>
+                    <max>100.0</max>
+                    <resolution>0.01</resolution>
+                </range>
+            </lidar>
+            <topic>/scan</topic>
+            <frame_id>lidar_link</frame_id>
+        </sensor>
+    </gazebo>
     <gazebo>
+        <plugin
+            filename="gz-sim-sensors-system"
+            name="gz::sim::systems::Sensors">
+            <render_engine>ogre</render_engine>
+        </plugin>
         <plugin name="gz::sim::systems::DiffDrive" filename="gz-sim-diff-drive-system">
             <left_joint>left_wheel_1_joint</left_joint>
